File: rp2040DVI/rp2040DVI/rp2040DVI.kicad_pcb (KiCad board)
At the start: 4 copper layers, 62.7 x 30 mm, 73 parts, among them J1 HDMI_A, J2 USB_C_Receptacle_USB2.0, J3 CONUFL001-SMD-T, J5 Micro_SD_Card_Det2, SW1 SW_Push, SW3 SW_Push, U1 NCP1117-3.3_SOT223, U2 LSM6DSOXTR, U3 W25Q128JVS, U4 RP2040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

Commit message: added other designs
Parts:
- BOOT JUMPER: renamed from JP1
- renumbered SW3 to BOOT, SW1 to RESET
Other:
- board text added: "ANTENNA"
- board text added: "HDMI"
- board text added: "M3B"
- board text added: "SD-CARD"
- board text added: "USB-C"
