File: rp2040DVI/rp2040DVI/rp2040DVI.kicad_sch (KiCad schematic)
At the start: 75 parts, among them J1 HDMI_A, J2 USB_C_Receptacle_USB2.0, J3 CONUFL001-SMD-T, J5 Micro_SD_Card_Det2, SW1 SW_Push, SW3 SW_Push, U1 NCP1117-3.3_SOT223, U2 LSM6DSOXTR, U3 W25Q128JVS, U4 RP2040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

Commit message: added other designs
Changed lines of the file:
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@@
     (effects (font (size 2.54 2.54)) (justify left bottom))
   )
-  (text "USB-C" (at 15.24 20.32 0)
+  (text "USB-C" (at 16.51 20.32 0)
     (effects (font (size 2.54 2.54)) (justify left bottom))
   )
